Commit message: Ajout d'une caméra sur la simulation

File: src/arcl_simulation/urdf/robot_omni.urdf (robot description, URDF)
Before this commit: robot robot_omni, 8 links, 7 joints
Links:
- added link camera
- added link camera_optical
- link chassis: geometry collision box size=0.03 0.06 0.12; collision box size=0.2 0.2 0.05
Joints:
- added joint camera_joint: type fixed, parent base_link, child camera, origin xyz=0.11 0 0.2025 rpy=0 0.2 0
- added joint camera_optical_joint: type fixed, parent camera, child camera_optical, origin xyz=0 0 0 rpy=-1.5708 0 -1.5708

Commit message: Correction carton aruco de simu et algo de centrage

File: src/arcl_simulation/urdf/robot_omni.urdf (robot description, URDF)
Before this commit: robot robot_omni, 10 links, 9 joints
Links:
- link chassis: geometry collision box size=0.02 0.05 0.028; collision box size=0.2 0.2 0.05
Joints:
- joint camera_joint: origin xyz=0.11 0 0.2025 rpy=0 0.2 0 -> xyz=0.11 0 0.0855 rpy=0 0 0

Commit message: Ajout d'une mécanique pour tourner les cartons

File: src/arcl_simulation/urdf/robot_omni.urdf (robot description, URDF)
Before this commit: robot robot_omni, 10 links, 9 joints
Links:
- added link ascenseur, mass 0.2; visual box size=0.006 0.1 0.014; visual box size=0.008 0.016 0.02
- added link poignet, mass 0.15; collision cylinder length=0.01 radius=0.015; collision cylinder length=0.01 radius=0.015
- link chassis: geometry collision box size=0.02 0.05 0.028; collision box size=0.2 0.2 0.05
Joints:
- added joint ascenseur_joint: type prismatic, parent chassis, child ascenseur, origin xyz=0 0 0, axis 0 0 1, limit lower=0 upper=0.12 effort=50 velocity=0.1
- added joint poignet_joint: type revolute, parent ascenseur, child poignet, origin xyz=0.106 0 0.121, axis 1 0 0, limit lower=0 upper=1.5708 effort=5 velocity=2
